File: Electronics/Ball MIll/Ball MIll.kicad_pcb (KiCad board)
At the start: 2 copper layers, 25 x 35 mm, 9 parts, among them J1 Jack-DC, J2 Conn_01x01, J3 Conn_01x01, J4 Conn_01x01

Commit message: podated pcb
Connections:
- J3 pad 1: Net-(F1-Pad1) -> Net-(J1-Pad2)
Other:
- board text added: "12V"
- board text added: "L GND"
- board text added: "M GND"
- board text removed: "GND"
- board text removed: "LED"
- board text removed: "M 12V"
